Commit message: Added control files

File: Proyecto/astromech/src/astromech_description/urdf/astromech.xacro (robot description, xacro)
@@ -27,5 +27,5 @@
     </visual>
     <collision name='caster_collision'>
-      <origin rpy="0 0 0" xyz="-0.007115 0 0.001085"/>
+      <origin rpy="0 0 0" xyz="-0.007115 0 0.0005"/>
       <geometry>
         <sphere radius="0.001385"/>
@@ -43,7 +43,19 @@
     </collision>
     <visual name='caster_visual'>
-      <origin rpy="0 0 0" xyz="-0.007115 0 0.001085"/>
+      <origin rpy="0 0 0" xyz="-0.007115 0 0.0005"/>
       <geometry>
         <sphere radius="0.001385"/>
+      </geometry>
+    </visual>
+    <collision name='back_leg_collision'>
+      <origin rpy="0 0.97 0" xyz="-0.005 0 0.004"/>
+      <geometry>
+        <box size="0.003 0.0007 0.01135"/>
+      </geometry>
+    </collision>
+    <visual name='back_leg_visual'>
+      <origin rpy="0 0.97 0" xyz="-0.005 0 0.004"/>
+      <geometry>
+        <box size="0.003 0.0007 0.01135"/>
       </geometry>
     </visual>
@@ -124,5 +136,5 @@
   </joint>
   <joint type="continuous" name="left_wheel_hinge">
-    <origin xyz="0 -0.0027 0" rpy="0 0 0"/>
+    <origin xyz="0.009 0.00257 0.000385" rpy="0 0 0"/>
     <child link="left_wheel"/>
     <parent link="chassis"/>
@@ -132,5 +144,5 @@
   </joint>
   <joint type="continuous" name="right_wheel_hinge">
-    <origin xyz="0 0.0027 0" rpy="0 0 0"/>
+    <origin xyz="0.009 0.00257 0.000385" rpy="0 0 0"/>
     <child link="right_wheel"/>
     <parent link="chassis"/>

Commit message: Optimizacion de la transmision

File: Proyecto/astromech/src/astromech_description/urdf/astromech.xacro (robot description, xacro)
@@ -3,9 +3,9 @@
   <xacro:include filename="$(find astromech_description)/urdf/astromech.gazebo" />
   <!--xacro:include filename="$(find astromech_description)/urdf/materials.xacro" /-->
-  <xacro:include filename="$(find astromech_description)/urdf/macros.xacro"/>
+  <!--xacro:include filename="$(find astromech_description)/urdf/macros.xacro"/-->
   <link name='chassis'>
-    <pose>0 0 0.0081 0 0 0</pose>
+    <pose>0 0 0.0081 0 0 0</pose >
     <inertial>
-      <mass value="4"/>
+      <mass value="1"/>
       <origin xyz="0.0 0 0.0081" rpy=" 0 0 0"/>
       <inertia
@@ -16,4 +16,5 @@
     </inertial>
     <collision name='collision'>
+      <origin xyz="0 0 0.0081" rpy=" 0 0 0"/>
       <geometry>
         <box size="0.003 0.00687 0.0032"/>
@@ -80,5 +81,5 @@
     <!--origin xyz="0 -188 0.035" rpy="0 1.5707 1.5707"/-->
     <collision name="collision">
-      <origin rpy="0 1.5707 1.5707" xyz="0.009 -0.00257 0.000385"/>
+      <origin rpy="0 1.5707 1.5707" xyz="0 0 0"/>
       <geometry>
         <cylinder length=".001" radius=".001385"/>
@@ -86,5 +87,5 @@
     </collision>
     <visual name="left_wheel_visual">
-      <origin rpy="0 1.5707 1.5707" xyz="0.009 -0.00257 0.000385"/>
+      <origin rpy="0 1.5707 1.5707" xyz="0 0 0"/>
       <geometry>
         <cylinder length=".001" radius=".001385"/>
@@ -92,5 +93,5 @@
     </visual>
     <inertial>
-      <origin rpy="0 1.5707 1.5707" xyz="0.009 -0.00257 0.000385"/>
+      <origin rpy="0 1.5707 1.5707" xyz="0 0 0"/>
       <mass value="0.001"/>
       <cylinder_inertia m="0.01" r="0.001385" h="0.001"/>
@@ -104,5 +105,5 @@
     <!--origin xyz="0 188 0.035" rpy="0 1.5707 1.5707"/-->
     <collision name="collision">
-      <origin rpy="0 1.5707 1.5707" xyz="0.009 0.00257 0.000385"/>
+      <origin rpy="0 1.5707 1.5707" xyz="0 0 0"/>
       <geometry>
         <cylinder length=".001" radius=".001385"/>
@@ -110,5 +111,5 @@
     </collision>
     <visual name="right_wheel_visual">
-      <origin rpy="0 1.5707 1.5707" xyz="0.009 0.00257 0.000385"/>
+      <origin rpy="0 1.5707 1.5707" xyz="0 0 0"/>
       <geometry>
         <cylinder length=".001" radius=".001385"/>
@@ -116,5 +117,5 @@
     </visual>
     <inertial>
-      <origin rpy="0 1.5707 1.5707" xyz="0.009 0.00257 0.000385"/>
+      <origin rpy="0 1.5707 1.5707" xyz="0 0 0"/>
       <mass value="0.001"/>
       <cylinder_inertia m="0.01" r="0.001385" h="0.001"/>
@@ -136,5 +137,5 @@
   </joint>
   <joint type="continuous" name="left_wheel_hinge">
-    <origin xyz="0.009 0.00257 0.000385" rpy="0 0 0"/>
+    <origin xyz="0.009 -0.00447 0.000385" rpy="0 0 0"/>
     <child link="left_wheel"/>
     <parent link="chassis"/>
@@ -144,5 +145,5 @@
   </joint>
   <joint type="continuous" name="right_wheel_hinge">
-    <origin xyz="0.009 0.00257 0.000385" rpy="0 0 0"/>
+    <origin xyz="0.009 0.00447 0.000385" rpy="0 0 0"/>
     <child link="right_wheel"/>
     <parent link="chassis"/>

Commit message: added camera functionality

File: Proyecto/astromech/src/astromech_description/urdf/astromech.xacro (robot description, xacro)
@@ -4,4 +4,17 @@
   <!--xacro:include filename="$(find astromech_description)/urdf/materials.xacro" /-->
   <!--xacro:include filename="$(find astromech_description)/urdf/macros.xacro"/-->
+  <xacro:include filename="$(find astromech_description)/urdf/astromech.cameraplugin.xacro" />
+  <!--xacro:include filename="$(find astromech_description)/urdf/materials.xacro" /-->
+  <xacro:include filename="$(find astromech_description)/urdf/macros.xacro"/>
+  <xacro:property name="camera_size" value="0.02"/>
+  <xacro:property name="camera_origin_x" value="0.065"/>
+  <xacro:property name="camera_origin_y" value="0"/>
+  <xacro:property name="camera_origin_z" value="0.025"/>
+	<xacro:macro name="default_inertial" params="mass">
+    <inertial>
+      <mass value="${mass}"/>
+      <inertia ixx="1.0" ixy="0.0" ixz="0.0" iyy="1.0" iyz="0.0" izz="1.0"/>
+    </inertial>
+  </xacro:macro>
   <link name='chassis'>
     <pose>0 0 0.0081 0 0 0</pose >
@@ -152,3 +165,23 @@
     <joint_properties damping="0.0" friction="0.0"/>
   </joint>
+<!--Camera-->
+  <link name="camera">
+    <visual>
+      <geometry>
+        <box size="${camera_size} ${camera_size} ${camera_size}"/>
+      </geometry>
+      <material name="blue"/>
+    </visual>
+    <collision>
+      <geometry>
+        <box size="${camera_size} ${camera_size} ${camera_size}"/>
+      </geometry>
+    </collision>
+    <xacro:default_inertial mass="0.02"/>
+  </link>
+  <joint name="camera_joint" type="fixed">
+    <origin xyz="${camera_origin_x} ${camera_origin_y} ${camera_origin_z}" rpy="0 0 0"/>
+    <parent link="chassis"/>
+    <child link="camera"/>
+  </joint>
 </robot>
